Commit message: first commit

File: vrx_gazebo/worlds/example_course.world.xacro (robot description, xacro)
@@ -56,4 +56,68 @@
       <pose>-420 295 0 0 0 -2.04</pose>
     </include>
+    <include>
+      <uri>model://tower</uri>
+      <pose>-450 370 -156 1.5708 0 0</pose>
+    </include>
+   <include>
+      <uri>model://passenger_fleet</uri>
+      <pose>-850 500 0 0 0 -3.5</pose>
+   </include>
+   <include>
+      <uri>model://baltica</uri>
+      <pose>-700 500 0 0 0 0</pose>
+   </include>
+   <include>
+      <uri>model://jet_ski</uri>
+      <pose>-500 220 0 0 0 0</pose>
+   </include>
+   <include>
+      <uri>model://sailing_boat</uri>
+      <pose>-650 300 0 0 0 1.5708</pose>
+   </include>
+   <include>
+      <uri>model://maintenance_fleet</uri>
+      <pose>-650 -20 0 0 0 1.5708</pose>
+   </include>
+   <include>
+      <uri>model://bullet</uri>
+      <pose>-550 200 0 0 0 3.14</pose>
+   </include>
+   <include>
+      <uri>model://yacht_v1</uri>
+      <pose>-450 -15 0 0 0 0</pose>
+   </include>
+   <include>
+      <uri>model://yacht_v2</uri>
+      <pose>-300 -30 0 0 0 3.14</pose>
+   </include>
+   <include>
+      <uri>model://yacht_v3</uri>
+      <pose>-200 -5 0 0 0 3.14</pose>
+   </include>
+   <include>
+      <uri>model://navigation_buoys0</uri>
+      <pose>-700 400 0 0 0 0</pose>
+    </include>
+   <include>
+      <uri>model://navigation_buoys1</uri>
+      <pose>-700 420 0 0 0 0</pose>
+   </include>
+   <include>
+      <uri>model://broken_bridge</uri>
+      <pose>-760 320 0 0 0 0</pose>
+   </include>
+   <include>
+      <uri>model://person_standing</uri>
+      <pose>-522 172 0 0 0 3.14</pose>
+   </include>
+   <include>
+      <uri>model://person_walking</uri>
+      <pose>-512 172 0 0 0 -1.5708</pose>
+   </include>
+   <include>
+      <uri>model://aruco_visual_marker_0</uri>
+      <pose>-532 172 0.1 0 0 0</pose>
+   </include>
   </world>
 </sdf>

File: wamv_gazebo/urdf/components/wamv_camera.xacro (robot description, xacro)
@@ -110,5 +110,5 @@
     <!-- Sensor post to sensor post arm joint -->
     <joint name="${namespace}/${name}_post_to_${name}_post_arm_joint" type="fixed">
-      <origin xyz="${post_to_post_arm_x} 0 ${z-post_z-post_arm_to_camera_z}" rpy="0 0 0" />
+      <origin xyz="${post_to_post_arm_x} 0 ${z-post_z-post_arm_to_camera_z}" rpy="0 ${-pi/12} 0" />
       <parent link="${namespace}/${name}_post_link" />
       <child link="${namespace}/${name}_post_arm_link" />
@@ -135,8 +135,9 @@
 	</xacro:if>
         <camera name="${name}_camera">
-          <horizontal_fov>1.3962634</horizontal_fov>
+          <!--horizontal_fov>1.3962634</horizontal_fov-->
+          <hfov>45</hfov>
           <image>
-            <width>1280</width>
-            <height>720</height>
+            <width>960</width>
+            <height>600</height>
             <format>R8G8B8</format>
           </image>
@@ -162,8 +163,8 @@
           <frameName>${namespace}/${name}_link_optical</frameName>
           <hackBaseline>0.07</hackBaseline>
-          <distortionK1>0.0</distortionK1>
-          <distortionK2>0.0</distortionK2>
-          <distortionK3>0.0</distortionK3>
-          <distortionT1>0.0</distortionT1>
+          <distortionK1>-0.015435</distortionK1>
+          <distortionK2>0.123584</distortionK2>
+          <distortionK3>-0.003953</distortionK3>
+          <distortionT1>0.005400</distortionT1>
           <distortionT2>0.0</distortionT2>
         </plugin>

File: wamv_gazebo/urdf/wamv_gazebo.urdf.xacro (robot description, xacro)
@@ -131,9 +131,11 @@
       <xacro:include filename="$(find wamv_description)/urdf/cpu_cases.xacro" />
       <xacro:cpu_cases position="-0.15 0 1.53" orientation="0 0 0"/>
-      <!-- Add a stereo camera pair -->
-      <xacro:wamv_camera name="front_left_camera" y="0.1" x="0.75" P="${radians(15)}" />
-      <xacro:wamv_camera name="front_right_camera" y="-0.1" x="0.75" P="${radians(15)}" />
-      <!-- Add a camera facing right -->
-      <xacro:wamv_camera name="middle_right_camera" y="-0.45" P="${radians(15)}" Y="${radians(-90)}" post_Y="${radians(-90)}" />
+      <!-- Add a front camera -->
+      <xacro:wamv_camera name="front_camera" y="0.0" x="0.75" P="${radians(15)}" />
+      <!-- Add side cameras -->
+      <xacro:wamv_camera name="right_camera" y="-0.45" P="${radians(15)}" Y="${radians(-90)}" post_Y="${radians(-90)}" />
+      <xacro:wamv_camera name="left_camera" y="0.45" P="${radians(15)}" Y="${radians(90)}" post_Y="${radians(90)}" />
+      <!-- Add a rear camera -->
+      <xacro:wamv_camera name="rear_camera" y="0.0" x="-0.95" P="${radians(15)}" Y="${radians(-180)}" post_Y="${radians(-180)}"/>
       <!-- Add simulated GPS -->
       <xacro:wamv_gps name="gps_wamv" x="-0.85" />

File: wave_gazebo/world_models/ocean_waves/model.xacro (robot description, xacro)
@@ -17,6 +17,6 @@
 -->
 <world xmlns:xacro="http://ros.org/wiki/xacro">
-  <xacro:macro name="ocean_waves" params="gain:=0.1 period:=5
-                     direction_x:=1.0 direction_y:=0.0
+  <xacro:macro name="ocean_waves" params="gain:=0.2 period:=5
+                     direction_x:=1.0 direction_y:=1.0
                      angle:=0.4 scale:=1.5">
   <model name='ocean_waves'>
@@ -28,5 +28,5 @@
       <cell_count>50 50</cell_count>
       <wave>
-				<model>PMS</model>
+        <model>PMS</model>
         <period>${period}</period>
         <number>3</number>
